File: mediapad.kicad_pcb (KiCad board)
At the start: 2 copper layers, 66.7 x 88.1 mm, 47 parts, among them U1 ATmega32U4-AU, Y1 16MHz

Commit message: updated final pcb design
Parts:
- added G***: LOGO, mediapad:vinyl, F.Cu at (139.7, 68.4)
- added H5: MountingHole, MountingHole:MountingHole_2.2mm_M2, F.Cu at (122.2, 68.3)
- added H6: MountingHole, MountingHole:MountingHole_2.2mm_M2, F.Cu at (157.2, 68.3)
Routing:
- net GND: track 505.7 -> 485.5 mm, vias 1 -> 2
- net +5V: track 404.2 -> 407.4 mm
Other:
- board text added: "Designed by Noah L github.com/null-ll"
- board text added: "JLCJLCJLCJLC"
